Commit message: Add files via upload

File: zed_bot/urdf/robot_1.xacro (robot description, xacro)
@@ -15,7 +15,7 @@
         <visual>
             <geometry>
-                <box size="0.45 0.2 0.165" />
+                <box size="0.45 0.25 0.17" />
             </geometry>
-            <origin xyz="0.2 0 0.1" rpy="0 0 0" />
+            <origin xyz="0.2 0 0.0" rpy="0 0 0" />
             <material name="green" />
         </visual>
@@ -26,5 +26,5 @@
         <parent link="base_link" />
         <child link= "zed_camera_link" />
-        <origin xyz="0.35 0.05 0.3" rpy="0 0 0" />
+        <origin xyz="0.35 0.05 0.35" rpy="0 0 0" />
     </joint>
 </robot>

Commit message: Add files via upload

File: zed_bot/urdf/robot_1.xacro (robot description, xacro)
@@ -26,5 +26,5 @@
         <parent link="base_link" />
         <child link= "zed_camera_link" />
-        <origin xyz="0.35 0.05 0.35" rpy="0 0 0" />
+        <origin xyz="0.35 0.05 0.6" rpy="0 0 0" />
     </joint>
 </robot>

Commit message: Add files via upload

File: zed_bot/urdf/robot_1.xacro (robot description, xacro)
@@ -21,10 +21,10 @@
         </visual>
     </link>
-    <link name="zed_camera_link" />
+    <link name="/support_frame" />
     <!-- Joints -->
     <joint name="zed_camera_link_joint" type="fixed">
         <parent link="base_link" />
-        <child link= "zed_camera_link" />
-        <origin xyz="0.35 0.05 0.6" rpy="0 0 0" />
+        <child link= "/support_frame" />
+        <origin xyz="0.35 0.0 0.58" rpy="0 0 0" />
     </joint>
 </robot>
